Commit message: update robot urdf with lidar working

File: src/step_01_robot_description/xacro_agv/agv_urdf.xacro (robot description, xacro)
@@ -13,4 +13,5 @@
     <xacro:include filename="$(find step_01_robot_description)/xacro_agv/lidar.xacro"/>
     <xacro:include filename="$(find step_01_robot_description)/xacro_agv/imu.xacro"/>
+    <xacro:include filename="$(find step_01_robot_description)/control/agv.gazebo"/>
     <!-- build robot -->
     <xacro:base_link/>

File: src/step_01_robot_description/xacro_agv/base_link.xacro (robot description, xacro)
@@ -15,6 +15,6 @@
           <mesh filename="package://step_01_robot_description/meshes/base_link.STL" />
         </geometry>
-        <material name="grey">
-          <color rgba="0.79 0.82 0.93 1" />
+        <material name="Blue">
+          <color rgba="0 0 1 1" />
         </material>
       </visual>

File: src/step_01_robot_description/xacro_agv/caster_behind_left.xacro (robot description, xacro)
@@ -18,6 +18,6 @@
           <mesh filename="package://step_01_robot_description/meshes/MT_behind_left.STL" />
         </geometry>
-        <material name="grey">
-          <color rgba="0.69 0.66 0.63 1" />
+        <material name="red">
+          <color rgba="1 0 0 1" />
         </material>
       </visual>

File: src/step_01_robot_description/xacro_agv/caster_behind_right.xacro (robot description, xacro)
@@ -18,6 +18,6 @@
           <mesh filename="package://step_01_robot_description/meshes/MT_behind_right.STL" />
         </geometry>
-        <material name="">
-          <color rgba="0.690196078431373 0.658823529411765 0.63921568627451 1" />
+        <material name="red">
+          <color rgba="1 0 0 1" />
         </material>
       </visual>

File: src/step_01_robot_description/xacro_agv/caster_up_left.xacro (robot description, xacro)
@@ -20,6 +20,6 @@
           <mesh filename="package://step_01_robot_description/meshes/MT_up_left.STL"/>
         </geometry>
-        <material name="caster_gray">
-          <color rgba="0.69 0.66 0.64 1"/>
+        <material name="red">
+          <color rgba="1 0 0 1"/>
         </material>
       </visual>

File: src/step_01_robot_description/xacro_agv/caster_up_right.xacro (robot description, xacro)
@@ -20,6 +20,6 @@
           <mesh filename="package://step_01_robot_description/meshes/MT_up_right.STL"/>
         </geometry>
-        <material name="grey">
-          <color rgba="0.690196078431373 0.658823529411765 0.63921568627451 1"/>
+        <material name="red">
+          <color rgba="1 0 0 1"/>
         </material>
       </visual>

File: src/step_01_robot_description/xacro_agv/lidar.xacro (robot description, xacro)
@@ -35,28 +35,31 @@
     <!-- Plugin cho Gazebo -->
     <gazebo reference="laser">
-      <sensor type="ray" name="lidar_sensor">
-        <pose>0 0 0 0 0 0</pose>
+      <sensor name="laser" type="gpu_lidar">
+        <topic>scan</topic>
+        <update_rate>10</update_rate>
+        <always_on>true</always_on>
         <visualize>true</visualize>
-        <update_rate>40</update_rate>
-        <ray>
+        <lidar>
           <scan>
             <horizontal>
               <samples>720</samples>
               <resolution>1</resolution>
-              <min_angle>-3.14</min_angle>
-              <max_angle>3.14</max_angle>
+              <min_angle>-3.14159</min_angle>
+              <max_angle>3.14159</max_angle>
             </horizontal>
+            <vertical>
+              <samples>1</samples>
+              <resolution>1</resolution>
+              <min_angle>0</min_angle>
+              <max_angle>0</max_angle>
+            </vertical>
           </scan>
           <range>
-            <min>0.10</min>
+            <min>0.2</min>
             <max>30.0</max>
-            <resolution>0.01</resolution>
+            <resolution>0.013</resolution>
           </range>
-          <noise>
-            <type>gaussian</type>
-            <mean>0.0</mean>
-            <stddev>0.01</stddev>
-          </noise>
-        </ray>
+        </lidar>
+        <gz_frame_id>laser</gz_frame_id>
       </sensor>
     </gazebo>

File: src/step_01_robot_description/xacro_agv/wheel_left.xacro (robot description, xacro)
@@ -13,6 +13,6 @@
           <mesh filename="package://step_01_robot_description/meshes/Wheel_left.STL" />
         </geometry>
-        <material name="">
-          <color rgba="0.792156862745098 0.819607843137255 0.933333333333333 1" />
+        <material name="Red">
+          <color rgba="1 0 0 1" />
         </material>
       </visual>

File: src/step_01_robot_description/xacro_agv/wheel_right.xacro (robot description, xacro)
@@ -14,5 +14,5 @@
         </geometry>
         <material name="">
-          <color rgba="0.792156862745098 0.819607843137255 0.933333333333333 1" />
+          <color rgba="1 0 0 1" />
         </material>
       </visual>

Commit message: Add IMU plugin and fix configs

File: src/step_01_robot_description/xacro_agv/agv_urdf.xacro (robot description, xacro)
@@ -25,6 +25,6 @@
     <xacro:imu/>
     <!-- chỉ include ros2_control khi chạy với Gazebo -->
-    <xacro:if value="$(arg use_gazebo)">
+    <!-- <xacro:if value="$(arg use_gazebo)">
         <xacro:include filename="$(find step_01_robot_description)/xacro_agv/ros2_control.xacro"/>
-    </xacro:if>
+    </xacro:if> -->
 </robot>

File: src/step_01_robot_description/xacro_agv/imu.xacro (robot description, xacro)
@@ -2,5 +2,5 @@
 <robot xmlns:xacro="http://www.ros.org/wiki/xacro">
     <xacro:macro name="imu" params="">
-        <link name="imu_link">
+        <link name="imu">
             <inertial>
                 <mass value="0.01"/>
@@ -24,7 +24,17 @@
         <joint name="imu_joint" type="fixed">
             <parent link="base_link"/>
-            <child link="imu_link"/>
+            <child link="imu"/>
             <origin xyz="0.0005 0.00076 0.0359" rpy="0 0 0"/>
         </joint>
+        <!-- 2.5.2 IMU gz sim properties -->
+        <gazebo reference="imu">
+            <sensor name="imu" type="imu">
+                <topic>imu</topic>
+                <update_rate>30.0</update_rate>
+                <always_on>true</always_on>
+                <visualize>true</visualize>
+                <gz_frame_id>imu</gz_frame_id>
+            </sensor>
+        </gazebo>
     </xacro:macro>
 </robot>
